File: main.brd (EAGLE design)
At the start: 58.4 x 31.8 mm, 23 parts, among them IC1 LM358N, IC2 LM358N, IC3 7805TV

Commit message: Add real board photo
Parts:
- moved U$2 0.57 mm to (19.3, 33.3)
Changed lines of the file:
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@@
 <drawing>
 <settings>
-<setting alwaysvectorfont="yes"/>
+<setting alwaysvectorfont="no"/>
 <setting verticaltext="up"/>
 </settings>
@@
 </element>
 <element name="U$1" library="random" package="XT30" value="XT30" x="11.43" y="29.21" smashed="yes" rot="R270"/>
-<element name="U$2" library="random" package="LOGO" value="" x="19.812" y="33.528" smashed="yes"/>
+<element name="U$2" library="random" package="LOGO" value="" x="19.304" y="33.274" smashed="yes"/>
 </elements>
 <signals>
